File: carte-sonars-gros-robot-2019/carte-sonars-gros-robot-2019.kicad_pcb (KiCad board)
At the start: 2 copper layers, 110 x 55 mm, 34 parts, among them SW1 SW_Push_Dual, U1 MCP2515-18Lead, U2 2x16BUSconnector, U3 MCP2551-I/P, Y1 16MHz

Commit message: PCB completed
Other:
- net class Default: via_dia 0.6 -> 0.9; via_drill 0.4 -> 0.6
- board text added: "2019"
- board text added: "Romain"
- board text added: "V 1.0"
- board text removed: "Romain 2019"
Changed lines of the file:
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@@
     (links 106)
     (no_connects 0)
-    (area 86.924999 91.924999 197.075001 147.075001)
+    (area 86.924999 84.674999 197.902382 148.307)
     (thickness 1.6)
-    (drawings 13)
+    (drawings 15)
     (tracks 243)
     (zones 0)
@@
     (segment_width 0.2)
     (edge_width 0.15)
-    (via_size 0.6)
-    (via_drill 0.4)
+    (via_size 0.9)
+    (via_drill 0.6)
     (via_min_size 0.4)
     (via_min_drill 0.3)
@@
     (visible_elements FFFFFF7F)
     (pcbplotparams
-      (layerselection 0x00030_80000001)
+      (layerselection 0x01000_80000001)
       (usegerberextensions false)
       (excludeedgelayer true)
@@
       (outputformat 1)
       (mirror false)
-      (drillshape 1)
+      (drillshape 0)
       (scaleselection 1)
       (outputdirectory ""))
@@
     (clearance 0.2)
     (trace_width 0.7)
-    (via_dia 0.6)
-    (via_drill 0.4)
+    (via_dia 0.9)
+    (via_drill 0.6)
     (uvia_dia 0.3)
     (uvia_drill 0.1)
@@
       (net 3 /GNDL) (zone_connect 2))
   )
-  (gr_text "Robotik UTT" (at 89.154 114.046) (layer F.Cu)
+  (gr_text "V 1.0" (at 89.916 119.634) (layer F.Cu)
+    (effects (font (size 1.3 1.3) (thickness 0.3)) (justify left))
+  )
+  (gr_text 2019 (at 89.916 117.094) (layer F.Cu)
     (effects (font (size 1.5 1.5) (thickness 0.3)) (justify left))
   )
-  (gr_text "Romain\n2019" (at 90.17 120.396) (layer F.Cu)
+  (gr_text "Robotik UTT" (at 159.004 145.288) (layer F.Cu)
+    (effects (font (size 1.5 1.5) (thickness 0.3)) (justify left))
+  )
+  (gr_text Romain (at 89.916 114.3) (layer F.Cu)
     (effects (font (size 1.5 1.5) (thickness 0.3)) (justify left))
   )
@@
   (segment (start 116.078 120.65) (end 112.014 120.65) (width 0.4) (layer B.Cu) (net 5))
   (segment (start 117.602 122.174) (end 116.078 120.65) (width 0.4) (layer B.Cu) (net 5))
-  (via (at 117.602 122.174) (size 0.6) (drill 0.4) (layers F.Cu B.Cu) (net 5))
+  (via (at 117.602 122.174) (size 0.9) (drill 0.6) (layers F.Cu B.Cu) (net 5))
   (segment (start 139.7 122.174) (end 117.602 122.174) (width 0.4) (layer F.Cu) (net 5))
   (segment (start 141.986 119.888) (end 139.7 122.174) (width 0.4) (layer F.Cu) (net 5))
   (segment (start 141.986 110.998) (end 141.986 119.888) (width 0.4) (layer F.Cu) (net 5))
-  (via (at 141.986 110.998) (size 0.6) (drill 0.4) (layers F.Cu B.Cu) (net 5))
+  (via (at 141.986 110.998) (size 0.9) (drill 0.6) (layers F.Cu B.Cu) (net 5))
   (segment (start 144.824 108.16) (end 141.986 110.998) (width 0.4) (layer B.Cu) (net 5))
   (segment (start 139.72 143.72) (end 147.848 143.72) (width 0.4) (layer B.Cu) (net 5))
