File: carte-actionneurs-gros-robot-2019/carte-actionneurs-gros-robot-2019.sch (KiCad schematic (older format))
At the start: 1 part

Commit message: PCB completed
Parts:
- removed U?: 2x16BUSconnector, symbol 2x16BUSconnector
- added A1: Arduino_Nano, Arduino_nano:arduino_nano, symbol Arduino_Nano
- added C1, C2: 22pF, Capacitors_THT:C_Disc_D3.4mm_W2.1mm_P2.50mm, symbol C
- added C_5VL1: 100nF, Capacitors_THT:C_Disc_D3.4mm_W2.1mm_P2.50mm, symbol C
- added Cp_5VL1: 10µF, Capacitors_THT:CP_Radial_D5.0mm_P2.50mm, symbol CP
- added D_POWER1, D_RXCAN1, D_TXCAN1: LED, LEDs:LED_D3.0mm, symbol LED
- added J_BAU1: Conn_01x02_Male, Pin_Headers:Pin_Header_Straight_1x02_Pitch2.54mm, symbol Conn_01x02_Male
- added J_PinAnalog1, J_Stepper0, J_Stepper1: Conn_01x04_Male, Pin_Headers:Pin_Header_Straight_1x04_Pitch2.54mm, symbol Conn_01x04_Male
- added J_Servo0, J_Servo1: Conn_01x03_Male, Pin_Headers:Pin_Header_Straight_1x03_Pitch2.54mm, symbol Conn_01x03_Male
- added Pololu0, Pololu1: PololuA4988, lib:PololuA4988, symbol PololuA4988
- added R1: 15k, Resistors_THT:R_Axial_DIN0207_L6.3mm_D2.5mm_P7.62mm_Horizontal, symbol R
- added R_CAN1: 120R, Resistors_THT:R_Axial_DIN0207_L6.3mm_D2.5mm_P7.62mm_Horizontal, symbol R
- added R_POWER1, R_RXCAN1, R_TXCAN1: 680R, Resistors_THT:R_Axial_DIN0207_L6.3mm_D2.5mm_P7.62mm_Horizontal, symbol R
- added SW1: SW_Push_Dual, Buttons_Switches_THT:SW_TH_Tactile_Omron_B3F-10xx, symbol SW_Push_Dual
- added U1: MCP2515-18Lead, Housings_DIP:DIP-18_W7.62mm_Socket_LongPads, symbol MCP2515-18Lead
- added U2: 2x16BUSconnector, Pin_Headers:Pin_Header_Angled_2x16_Pitch2.54mm, symbol 2x16BUSconnector
- added U3: MCP2551-I/P, Housings_DIP:DIP-8_W7.62mm, symbol MCP2551-I/P
- added Y1: 16MHz, Crystals:Crystal_SMD_HC49-SD_HandSoldering, symbol Crystal
Connections:
- net 5VL: now also A1.27 (5V), C_5VL1.1, Cp_5VL1.1, D_POWER1.1 (K), J_BAU1.2 (Pin_2), Pololu0.10 (VDD), Pololu1.10 (VDD), R_RXCAN1.2, R_TXCAN1.2, U1.18 (Vdd), U2.17 (5VL), U2.18, U3.3 (VDD)
- net BAU: now also J_BAU1.1 (Pin_1), U2.31 (BAU), U2.32
- net CANH: now also R_CAN1.1, U2.25 (CANH), U2.26, U3.7 (CANH)
- net CANL: now also R_CAN1.2, U2.27 (CANL), U2.28, U3.6 (CANL)
- new net: A1.10 (D7), J_Servo1.3 (Pin_3)
- new net: A1.11 (D8), J_Servo1.2 (Pin_2)
- new net: A1.12 (D9), J_Servo1.1 (Pin_1)
- new net: A1.23 (AD4/D18), J_PinAnalog1.4 (Pin_4)
- new net: A1.24 (AD5/D19), J_PinAnalog1.3 (Pin_3)
- new net: A1.25 (AD6), J_PinAnalog1.2 (Pin_2)
- new net: A1.26 (AD7), J_PinAnalog1.1 (Pin_1)
- new net: A1.5 (D2), J_Servo0.3 (Pin_3)
- new net: A1.6 (D3), J_Servo0.2 (Pin_2)
- new net: A1.7 (D4), J_Servo0.1 (Pin_1)
- new net: C1.1, U1.7 (OSC2), Y1.1
- new net: C2.1, U1.8 (OSC1), Y1.2
- new net: D_TXCAN1.2 (A), R_TXCAN1.1
- new net: R1.1, U3.8 (Rs)
- new net: D_RXCAN1.2 (A), R_RXCAN1.1
- new net: D_POWER1.2 (A), R_POWER1.1
- new net: J_Stepper0.1 (Pin_1), Pololu0.11 (1B)
- new net: J_Stepper0.2 (Pin_2), Pololu0.12 (1A)
- new net: J_Stepper0.3 (Pin_3), Pololu0.13 (2A)
- new net: J_Stepper0.4 (Pin_4), Pololu0.14 (2B)
- new net: Pololu0.5 (RST), Pololu0.6 (SLP)
- new net: J_Stepper1.1 (Pin_1), Pololu1.11 (1B)
- new net: J_Stepper1.2 (Pin_2), Pololu1.12 (1A)
- new net: J_Stepper1.3 (Pin_3), Pololu1.13 (2A)
- new net: J_Stepper1.4 (Pin_4), Pololu1.14 (2B)
- new net: Pololu1.5 (RST), Pololu1.6 (SLP)
- new net +12AX: Pololu0.16 (VMOT), Pololu1.16 (VMOT), U2.10, U2.9 (+12AX)
- new net +5P: U2.21 (+5P), U2.22
- new net 3V3: A1.17 (3V3)
- new net DIR0: A1.20 (AD1/D15), Pololu0.8 (DIR)
- new net DIR1: A1.22 (AD3/D17), Pololu1.8 (DIR)
- new net EN0: A1.8 (D5), Pololu0.1 (EN)
- new net EN1: A1.9 (D6), Pololu1.1 (EN)
- new net GNDAX: A1.29 (GND), A1.4 (GND), C1.2, C2.2, C_5VL1.2, Cp_5VL1.2, Pololu0.15 (GND), Pololu0.9 (GND), Pololu1.15 (GND), Pololu1.9 (GND), R1.2, R_POWER1.2, SW1.4, U1.9 (Vss), U2.11 (GNDAX), U2.12, U2.19 (GNDL), U2.20, U2.23 (GNDP), U2.24, U3.2 (VSS)
- new net MISO1: A1.15 (D12), U1.15 (SO)
- new net MOSI1: A1.14 (D11), U1.14 (SI)
- new net RST: A1.3 (RESET), SW1.1, U1.17 (RESET)
- new net RXCAN1: D_RXCAN1.1 (K), U1.2 (RXCAN), U3.4 (RXD)
- new net SCK1: A1.16 (D13), U1.13 (SCK)
- new net SS1: A1.13 (D10), U1.16 (CS)
- new net STEP0: A1.19 (AD0/D14), Pololu0.7 (STEP)
- new net STEP1: A1.21 (AD2/D16), Pololu1.7 (STEP)
- new net TXCAN1: D_TXCAN1.1 (K), U1.1 (TXCAN), U3.1 (TXD)
